File: snare-drum.kicad_pcb (KiCad board)
At the start: 2 copper layers, 11 parts, among them J1 Conn_02x05_Odd_Even

Commit message: v0 ready
Parts:
- added C10: 33n, Capacitor_SMD:C_0805_2012Metric, F.Cu at (67.3, 81.0)
- added C11: 2.2n, Capacitor_SMD:C_0805_2012Metric, F.Cu at (67.1, 20.3)
- added C12: 2.2n, Capacitor_SMD:C_0805_2012Metric, F.Cu at (68.8, 27.9)
- added C13: 1n, Capacitor_SMD:C_0805_2012Metric, F.Cu at (66.3, 27.9)
- added C14: 1n, Capacitor_SMD:C_0805_2012Metric, F.Cu at (63.8, 27.9)
- added C15: 10n, Capacitor_SMD:C_0805_2012Metric, F.Cu at (63.8, 33.2)
- added C16: 470n, Capacitor_SMD:C_0805_2012Metric, F.Cu at (69.9, 46.5)
- added C3: 100n, Capacitor_SMD:C_0805_2012Metric, F.Cu at (71.4, 104.9)
- added C4: 100n, Capacitor_SMD:C_0805_2012Metric, F.Cu at (69.6, 67.3)
- added C5: 10n, Capacitor_SMD:C_0805_2012Metric, F.Cu at (62.7, 98.3)
- added C6: 33n, Capacitor_SMD:C_0805_2012Metric, F.Cu at (59.2, 72.9)
- added C7: 33n, Capacitor_SMD:C_0805_2012Metric, F.Cu at (59.2, 68.8)
- added C8: 470n, Capacitor_SMD:C_0805_2012Metric, F.Cu at (66.8, 85.1)
- added C9: 1u box, Capacitor_THT:C_Rect_L7.2mm_W7.2mm_P5.00mm_FKS2_FKP2_MKS2_MKP2, B.Cu at (60.2, 10.9)
- added D3: 1N4148, Diode_SMD:D_SOD-323_HandSoldering, F.Cu at (61.7, 104.9)
- added D4: 1N4148, Diode_SMD:D_SOD-323_HandSoldering, F.Cu at (62.7, 91.7)
- added D5: 1N4148, Diode_SMD:D_SOD-323_HandSoldering, F.Cu at (67.3, 23.6)
- added D6: 1N4148, Diode_SMD:D_SOD-323_HandSoldering, F.Cu at (69.9, 50.0)
- added D7: 1N4148, Diode_SMD:D_SOD-323_HandSoldering, F.Cu at (78.0, 50.0)
- added D8: 1N4148, Diode_SMD:D_SOD-323_HandSoldering, F.Cu at (82.6, 50.0)
- added D9: 1N4148, Diode_SMD:D_SOD-323_HandSoldering, F.Cu at (80.5, 47.5)
- added H10: gate, Eurorack:Mech-AudioJack-Hole-Input-Gate, F.Cu at (79.6, 182.7)
- added H11: accent, Eurorack:Mech-AudioJack-Hole-Input-CV, F.Cu at (79.6, 207.7)
- added H12: pitch, Eurorack:Mech-AudioJack-Hole-Input-CV, F.Cu at (79.6, 195.2)
- added H13: snappy, Eurorack:Mech-AudioJack-Hole-Input-CV, F.Cu at (79.6, 220.2)
- added H14: out, Eurorack:Mech-AudioJack-Hole-Output, F.Cu at (79.6, 234.7)
- added H5: decay, Eurorack:Mech-Potentiometer-Hole_level, F.Cu at (65.1, 168.7)
- added H6: attack, Eurorack:Mech-Potentiometer-Hole_level, F.Cu at (65.1, 194.7)
- added H7: pitch, Eurorack:Mech-Potentiometer-Hole_level, F.Cu at (65.1, 220.7)
- added H8: snappy, Eurorack:Mech-Potentiometer-Hole_level, F.Cu at (65.1, 142.7)
- added H9: pitch cv, Eurorack:Mech-LED-Hole-3mm, F.Cu at (83.1, 163.8)
- added J2: GATE, Eurorack:AudioJack2_Tayda_A-2566, F.Cu at (79.6, 60.9)
- added J3: ACCENT_CV, Eurorack:AudioJack2_Tayda_A-2566, F.Cu at (79.6, 85.9)
- added J4: PITCH_CV, Eurorack:AudioJack2_Tayda_A-2566, F.Cu at (79.6, 73.4)
- added J5: SNAPPY_CV, Eurorack:AudioJack2_Tayda_A-2566, F.Cu at (79.6, 98.4)
- added J6: OUT, Eurorack:AudioJack2_Tayda_A-2566, F.Cu at (79.6, 112.9)
- added Q1: BCM857, Package_SO:TSOP-6_1.65x3.05mm_P0.95mm, F.Cu at (65.8, 50.0)
- added Q2: BCM847, Package_SO:TSOP-6_1.65x3.05mm_P0.95mm, F.Cu at (62.5, 85.1)
- added Q3: BC547C, Package_TO_SOT_THT:TO-92_Inline_Wide, B.Cu at (66.5, 16.0)
- added Q4: BCM847, Package_SO:TSOP-6_1.65x3.05mm_P0.95mm, F.Cu at (62.7, 22.6)
- added R10: 1K, Resistor_SMD:R_0805_2012Metric, F.Cu at (59.2, 76.9)
- added R11: 910K, Resistor_SMD:R_0805_2012Metric, F.Cu at (62.7, 71.9)
- added R12: 330, Resistor_SMD:R_0805_2012Metric, F.Cu at (67.8, 117.6)
- added R13: 470, Resistor_SMD:R_0805_2012Metric, F.Cu at (62.2, 117.6)
- added R14: 47K, Resistor_SMD:R_0805_2012Metric, F.Cu at (71.4, 81.0)
- added R15: 47K, Resistor_SMD:R_0805_2012Metric, F.Cu at (62.7, 60.2)
- added R16: 470K, Resistor_SMD:R_0805_2012Metric, F.Cu at (59.2, 81.0)
- added R17: 47K, Resistor_SMD:R_0805_2012Metric, F.Cu at (71.9, 85.1)
- added R18: 27K, Resistor_SMD:R_0805_2012Metric, F.Cu at (69.4, 85.1)
- added R19: 1K, Resistor_SMD:R_0805_2012Metric, F.Cu at (67.3, 91.7)
- added R20: 100K, Resistor_SMD:R_0805_2012Metric, F.Cu at (62.7, 67.8)
- added R21: 100K, Resistor_SMD:R_0805_2012Metric, F.Cu at (62.7, 11.4)
- added R22: 100K, Resistor_SMD:R_0805_2012Metric, F.Cu at (62.7, 15.5)
- added R23: 22K, Resistor_SMD:R_0805_2012Metric, F.Cu at (62.7, 78.5)
- added R24: 1M, Resistor_SMD:R_0805_2012Metric, F.Cu at (62.7, 81.0)
- added R25: 1M, Resistor_SMD:R_0805_2012Metric, F.Cu at (58.4, 27.9)
- added R26: 100K, Resistor_SMD:R_0805_2012Metric, F.Cu at (61.2, 27.9)
- added R27: 22K, Resistor_SMD:R_0805_2012Metric, F.Cu at (68.8, 33.2)
- added R28: 22K, Resistor_SMD:R_0805_2012Metric, F.Cu at (61.2, 33.2)
- added R29: 22K, Resistor_SMD:R_0805_2012Metric, F.Cu at (65.8, 46.5)
- added R3: 39K, Resistor_SMD:R_0805_2012Metric, F.Cu at (65.3, 98.3)
- added R30: 10K, Resistor_SMD:R_0805_2012Metric, F.Cu at (66.3, 33.2)
- added R31: 33K, Resistor_SMD:R_0805_2012Metric, F.Cu at (64.8, 111.5)
- added R32: 1K, Resistor_SMD:R_0805_2012Metric, F.Cu at (67.3, 111.5)
- added R33: 10K, Resistor_SMD:R_0805_2012Metric, F.Cu at (78.0, 52.5)
- added R34: 10K, Resistor_SMD:R_0805_2012Metric, F.Cu at (82.6, 52.5)
- added R35: 10K, Resistor_SMD:R_0805_2012Metric, F.Cu at (80.5, 44.9)
- added R4: 33K, Resistor_SMD:R_0805_2012Metric, F.Cu at (67.8, 98.3)
- added R5: 100K, Resistor_SMD:R_0805_2012Metric, F.Cu at (70.4, 98.3)
- added R6: 100K, Resistor_SMD:R_0805_2012Metric, F.Cu at (61.7, 49.0)
- added R7: 22K, Resistor_SMD:R_0805_2012Metric, F.Cu at (61.7, 46.5)
- added R8: 120K, Resistor_SMD:R_0805_2012Metric, F.Cu at (61.7, 51.5)
- added R9: 10K, Resistor_SMD:R_0805_2012Metric, F.Cu at (62.7, 75.9)
- added RV1: B1K, Eurorack:Potentiometer_RV16AF-41-15R1, F.Cu at (65.1, 98.9)
- added RV2: B100K, Eurorack:Potentiometer_RV16AF-41-15R1, F.Cu at (65.1, 46.9)
- added RV3: B5K, Eurorack:Potentiometer_RV16AF-41-15R1, F.Cu at (65.1, 72.9)
- added RV4: 100K, Potentiometer_THT:Potentiometer_Bourns_3296W_Vertical, F.Cu at (82.2, 40.9)
- added RV5: B100K, Eurorack:Potentiometer_RV16AF-41-15R1, F.Cu at (65.1, 20.9)
- added U1: TL072, Package_SO:SOIC-8_3.9x4.9mm_P1.27mm, F.Cu at (66.3, 104.9)
- added U2: TL074, Package_SO:SO-14_3.9x8.65mm_P1.27mm, F.Cu at (69.4, 73.9)
- moved H3 225.8 mm to (81.1, 247.4)
- moved H4 218.3 mm to (61.1, 247.4)
- moved H2 112.4 mm to (81.1, 124.9)
- moved H1 110.6 mm to (61.1, 124.9)
- moved C2 49.5 mm to (74.5, 13.5), turned to 180 degrees
- moved D2 43.9 mm to (75.5, 16.8), turned to -90 degrees
- moved R1 38.6 mm to (76.5, 20.1), turned to 0 degrees
- moved R2 34.2 mm to (76.5, 22.6), turned to 0 degrees
- moved J1 32.4 mm to (79.8, 26.5), turned to 0 degrees
- moved D1 27.5 mm to (75.5, 26.0), turned to -90 degrees
- moved C1 18.7 mm to (72.0, 29.0), turned to 0 degrees
Routing:
- net -12V: track 14.7 -> 146.2 mm, vias 0 -> 2
- net +12V: track 14.2 -> 145.3 mm, vias 0 -> 3
- net GND: track 41.0 -> 159.2 mm, vias 0 -> 21
- net Net-(U1B--): track 0.00 -> 85.7 mm, vias 0 -> 3
- net Net-(Q4A-B1): track 0.00 -> 78.1 mm, vias 0 -> 2
- net Net-(U2B-+): track 0.00 -> 67.3 mm, vias 0 -> 1
- net Net-(D4-A): track 0.00 -> 63.1 mm
- net /GATE: track 0.00 -> 60.8 mm, vias 0 -> 1
- net Net-(C6-Pad2): track 0.00 -> 54.2 mm, vias 0 -> 3
- net Net-(D6-A): track 0.00 -> 45.9 mm
- net Net-(Q2A-B1): track 0.00 -> 43.6 mm
- net /SNAPPY_CV: track 0.00 -> 42.6 mm, vias 0 -> 1
- net Net-(R15-Pad2): track 0.00 -> 41.2 mm, vias 0 -> 1
- net Net-(Q2B-C2): track 0.00 -> 35.8 mm, vias 0 -> 1
- net /PITCH_CV: track 0.00 -> 34.4 mm
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- added copper zone on B.Cu, net /FACE
- added copper zone on F.Cu, net /FACE
- added copper zone on B.Cu, net GND
- added copper zone on F.Cu, net GND
Other:
- board outline added: 30 x 241 mm
- board text added: "snare"
- board text added: "thismatters/snare-drum/v0"

Commit message: add ident
Parts:
- added REF**: IDENT, Eurorack:Lot_Ident, F.Cu at (71.6, 21.2)
Changed lines of the file:
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@@
 		)
 	)
+	(footprint "Eurorack:Lot_Ident"
+		(layer "F.Cu")
+		(at 71.628 21.209)
+		(property "Reference" "REF**"
+			(at 0 -0.5 0)
+			(unlocked yes)
+			(layer "F.SilkS")
+			(hide yes)
+			(effects
+				(font
+					(size 1 1)
+					(thickness 0.1)
+				)
+			)
+		)
+		(property "Value" "IDENT"
+			(at -2.54 0 270)
+			(unlocked yes)
+			(layer "B.SilkS")
+			(effects
+				(font
+					(size 1 1)
+					(thickness 0.15)
+				)
+				(justify mirror)
+			)
+		)
+		(property "Datasheet" ""
+			(at 0 0 0)
+			(unlocked yes)
+			(layer "F.Fab")
+			(hide yes)
+			(effects
+				(font
+					(size 1 1)
+					(thickness 0.15)
+				)
+			)
+		)
+		(property "Description" ""
+			(at 0 0 0)
+			(unlocked yes)
+			(layer "F.Fab")
+			(hide yes)
+			(effects
+				(font
+					(size 1 1)
+					(thickness 0.15)
+				)
+			)
+		)
+		(attr smd)
+		(duplicate_pad_numbers_are_jumpers no)
+		(fp_poly
+			(pts
+				(xy 1.016 3.048) (xy 0.508 3.556) (xy 1.524 3.556)
+			)
+			(stroke
+				(width 0.1)
+				(type solid)
+			)
+			(fill yes)
+			(layer "B.SilkS")
+		)
+		(fp_text user "${REFERENCE}"
+			(at 0 2.5 0)
+			(unlocked yes)
+			(layer "F.Fab")
+			(effects
+				(font
+					(size 1 1)
+					(thickness 0.15)
+				)
+			)
+		)
+		(pad "" smd rect
+			(at -1.016 -2.032)
+			(size 1.2 1.4)
+			(layers "B.Cu" "B.Mask" "B.Paste")
+		)
+		(pad "" smd rect
+			(at -1.016 0)
+			(size 1.2 1.4)
+			(layers "B.Cu" "B.Mask" "B.Paste")
+		)
+		(pad "" smd rect
+			(at -1.016 2.032)
+			(size 1.2 1.4)
+			(layers "B.Cu" "B.Mask" "B.Paste")
+		)
+		(pad "" smd rect
+			(at 1.016 -2.032)
+			(size 1.2 1.4)
+			(layers "B.Cu" "B.Mask" "B.Paste")
+		)
+		(pad "" smd rect
+			(at 1.016 0)
+			(size 1.2 1.4)
+			(layers "B.Cu" "B.Mask" "B.Paste")
+		)
+		(pad "" smd rect
+			(at 1.016 2.032)
+			(size 1.2 1.4)
+			(layers "B.Cu" "B.Mask" "B.Paste")
+		)
+		(embedded_fonts no)
+	)
 	(footprint "Package_SO:TSOP-6_1.65x3.05mm_P0.95mm"
 		(layer "F.Cu")
@@
 		(tags "CP Radial series Radial pin pitch 2.50mm  diameter 5mm Electrolytic Capacitor")
 		(property "Reference" "C1"
-			(at -0.572888 -3.302 90)
+			(at -1.487288 -2.7432 90)
 			(layer "B.SilkS")
 			(effects
@@
 		(tags "CP Radial series Radial pin pitch 2.50mm  diameter 5mm Electrolytic Capacitor")
 		(property "Reference" "C2"
-			(at 2.983113 -3.556 90)
+			(at 3.897513 -2.7178 90)
 			(layer "B.SilkS")
 			(effects
